File: ECEN_4330/PROJECT_V2.brd (EAGLE design)
At the start: 160 x 100 mm, 32 parts

Commit message: Started routing pcb, Fixed some mistakes on the schematic, added note for BCD converter in code.
Parts:
- removed 7SEGDISPLAY:7SEG: 7_SEG, Fuckboiz:754-1460-5-ND
- removed 7SEGDISPLAY:7SEGLATCH: 74HC573N, Fuckboiz:DIL20
- removed 7SEGDISPLAY:R2, 7SEGDISPLAY:R3, 7SEGDISPLAY:R4, 7SEGDISPLAY:R5, 7SEGDISPLAY:R6, 7SEGDISPLAY:R7, 7SEGDISPLAY:R8, 7SEGDISPLAY:R9: 330, adafruit:0204/7
- removed CLOCK:CLK: XC269-ND, crystal:DIL08S
- removed KEYPAD1:KEYPAD: (no value), Fuckboiz:KEYPAD4X4
- removed MICROCONTROLLER1:C1: 10u, adafruit:C025-025X050
- removed MICROCONTROLLER1:DEMULTIPLEXER: 74AS573N, Fuckboiz:DIL20
- removed MICROCONTROLLER1:MICROCONTROLLER: 8051P, Fuckboiz:DIL40
- removed MICROCONTROLLER1:R1: 8.2k, rcl:0204/5
- removed MICROCONTROLLER1:RSTSWITCH: MOMENTARY-SWITCH-SPST-PTH-6.0MM, SparkFun-Switches:TACTILE_SWITCH_PTH_6.0MM
- removed POWERSP:J1: DCpowerjack, Fuckboiz:SPC4077
- removed POWERSP:LED1: (no value), adafruit:LED5MM
- removed POWERSP:R11: 1k, resistor:0204/7
- removed POWERSP:S1: (no value), Fuckboiz:SPDT_EG2355-ND
- added 7SEG:7SEG: 7_SEG, Fuckboiz:754-1460-5-ND
- added 7SEG:7SEGLATCH, MC:DEMULTIPLEXER: 74AS573N, Fuckboiz:DIL20
- added 7SEG:C1, ADC:C1, ADC:C2, C101, LCD:C1, LCD:C2, MC:C2, RAM:C1, RAM:C2, ROM:C1, ROM:C2, RTC:C1: 0.1uF, Fuckboiz:CAP-PTH-SMALL-KIT
- added 7SEG:R2, 7SEG:R3, 7SEG:R4, 7SEG:R5, 7SEG:R6, 7SEG:R7, 7SEG:R8, 7SEG:R9: 330, adafruit:0204/7
- added CLK:CLK: XC269-ND, crystal:DIL08S
- added KP:KEYPAD: (no value), Fuckboiz:KEYPAD4X4
- added MC:C1: 10u, adafruit:C025-025X050
- added MC:JPM: (no value), pinhead:1X05
- added MC:MICROCONTROLLER: 8051P, Fuckboiz:DIL40
- added MC:R1: 8.2k, rcl:0204/7
- added MC:RSTSWITCH: MOMENTARY-SWITCH-SPST-PTH-6.0MM, SparkFun-Switches:TACTILE_SWITCH_PTH_6.0MM
- added PWR:PWRFUSE: 2.5A, Fuckboiz:SHK20Q
- added PWR:PWRJACK: DCpowerjack, Fuckboiz:SPC4077
- added PWR:PWRLED: (no value), adafruit:LED5MM
- added PWR:R11: 1k, resistor:0204/7
- added PWR:S1: (no value), Fuckboiz:SPDT_EG2355-ND
- moved LCD:R10 357.1 mm to (212.1, 111.8), turned to 180 degrees
- moved RTC:RTC 351.7 mm to (47.0, 16.5), turned to 270 degrees
- moved CSLOGIC100 334.3 mm to (133.3, 55.9), turned to 270 degrees
- moved ADC:ADC 323.6 mm to (22.9, 6.35)
- moved LCD:IC1 319.1 mm to (193.0, 111.8)
- moved ADC:TEMPSENS 304.1 mm to (8.89, 27.9), turned to 270 degrees
- moved LCD:LCD 263.1 mm to (172.7, 188.0), turned to 180 degrees
- moved RAM:RAM2 231.3 mm to (63.5, 44.5)
- moved RAM:RAM1 165.3 mm to (63.5, 109.2)
- moved ROM:ROM2 121.4 mm to (26.7, 45.7)
- moved ROM:ROM1 54.6 mm to (26.7, 110.5)
Connections:
- net CHIPSELECT:N$1 renamed CS:N$1
- net CHIPSELECT:N$2 renamed CS:N$2
- net CHIPSELECT:N$3 renamed CS:N$3
- net CHIPSELECT:N$35 renamed CS:N$35
- net CHIPSELECT:N$4 renamed CS:N$4
- net N$10 renamed LCDCS
- net N$11 renamed COLORCS
- net N$12 renamed ROM1CS
- net N$13 renamed ROM2CS
- net N$14 renamed RAM2CS
- net N$15 renamed RAM1CS
- net N$8 renamed RTCCS
- net N$9 renamed ADCCS
- removed net 7SEGDISPLAY:N$10: 7SEGDISPLAY:7SEG.10, 7SEGDISPLAY:R8.2
- removed net 7SEGDISPLAY:N$11: 7SEGDISPLAY:7SEG.9, 7SEGDISPLAY:R7.2
- removed net 7SEGDISPLAY:N$12: 7SEGDISPLAY:7SEG.1, 7SEGDISPLAY:R6.2
- removed net 7SEGDISPLAY:N$13: 7SEGDISPLAY:7SEG.2, 7SEGDISPLAY:R5.2
- removed net 7SEGDISPLAY:N$14: 7SEGDISPLAY:7SEG.4, 7SEGDISPLAY:R4.2
- removed net 7SEGDISPLAY:N$3: 7SEGDISPLAY:7SEGLATCH.19, 7SEGDISPLAY:R2.1
- removed net 7SEGDISPLAY:N$33: 7SEGDISPLAY:7SEG.6, 7SEGDISPLAY:R3.2
- removed net 7SEGDISPLAY:N$4: 7SEGDISPLAY:7SEGLATCH.18, 7SEGDISPLAY:R3.1
- removed net 7SEGDISPLAY:N$43: 7SEGDISPLAY:7SEG.7, 7SEGDISPLAY:R2.2
- removed net 7SEGDISPLAY:N$44: 7SEGDISPLAY:7SEG.5, 7SEGDISPLAY:R9.2
- removed net 7SEGDISPLAY:N$45: 7SEGDISPLAY:7SEGLATCH.12, 7SEGDISPLAY:R9.1
- removed net 7SEGDISPLAY:N$5: 7SEGDISPLAY:7SEGLATCH.17, 7SEGDISPLAY:R4.1
- removed net 7SEGDISPLAY:N$6: 7SEGDISPLAY:7SEGLATCH.16, 7SEGDISPLAY:R5.1
- removed net 7SEGDISPLAY:N$7: 7SEGDISPLAY:7SEGLATCH.15, 7SEGDISPLAY:R6.1
- removed net 7SEGDISPLAY:N$8: 7SEGDISPLAY:7SEGLATCH.14, 7SEGDISPLAY:R7.1
- removed net 7SEGDISPLAY:N$9: 7SEGDISPLAY:7SEGLATCH.13, 7SEGDISPLAY:R8.1
- removed net CHIPSELECT:GND: CSLOGIC100.12
- removed net CHIPSELECT:VCC: CSLOGIC100.24
- removed net MICROCONTROLLER1:N$15: MICROCONTROLLER1:C1.2, MICROCONTROLLER1:MICROCONTROLLER.9, MICROCONTROLLER1:R1.2, MICROCONTROLLER1:RSTSWITCH.1
- removed net MICROCONTROLLER1:N$18: MICROCONTROLLER1:MICROCONTROLLER.10
- removed net MICROCONTROLLER1:N$19: MICROCONTROLLER1:MICROCONTROLLER.11
- removed net MICROCONTROLLER1:N$20: MICROCONTROLLER1:MICROCONTROLLER.12
- removed net MICROCONTROLLER1:N$21: MICROCONTROLLER1:MICROCONTROLLER.13
- removed net MICROCONTROLLER1:N$22: MICROCONTROLLER1:MICROCONTROLLER.14
- removed net MICROCONTROLLER1:N$31: MICROCONTROLLER1:MICROCONTROLLER.18
- removed net N$1: ADC:ADC.8, CSLOGIC100.7, MICROCONTROLLER1:MICROCONTROLLER.17, RAM:RAM1.22, RAM:RAM2.22, RTC:RTC.8
- removed net N$2: ADC:ADC.6, CSLOGIC100.6, MICROCONTROLLER1:MICROCONTROLLER.16, RAM:RAM1.27, RAM:RAM2.27, RTC:RTC.10
- removed net N$3: CSLOGIC100.2, MICROCONTROLLER1:MICROCONTROLLER.29
- removed net N$4: CSLOGIC100.8, MICROCONTROLLER1:MICROCONTROLLER.15
- removed net N$6: MICROCONTROLLER1:DEMULTIPLEXER.11, MICROCONTROLLER1:MICROCONTROLLER.30, RTC:RTC.3
- removed net N$7: 7SEGDISPLAY:7SEGLATCH.11, CSLOGIC100.23
- removed net POWERSP:N$30: POWERSP:S1.1
- removed net POWERSP:N$48: POWERSP:J1.3, POWERSP:S1.2
- removed net POWERSP:N$49: POWERSP:LED1.K, POWERSP:R11.2
- new net 7SEG:N$10: 7SEG:7SEG.10, 7SEG:R8.2
- new net 7SEG:N$11: 7SEG:7SEG.9, 7SEG:R7.2
- new net 7SEG:N$12: 7SEG:7SEG.1, 7SEG:R6.2
- new net 7SEG:N$13: 7SEG:7SEG.2, 7SEG:R5.2
- new net 7SEG:N$14: 7SEG:7SEG.4, 7SEG:R4.2
- new net 7SEG:N$3: 7SEG:7SEGLATCH.19, 7SEG:R2.1
- new net 7SEG:N$33: 7SEG:7SEG.6, 7SEG:R3.2
- new net 7SEG:N$4: 7SEG:7SEGLATCH.18, 7SEG:R3.1
- new net 7SEG:N$43: 7SEG:7SEG.7, 7SEG:R2.2
- new net 7SEG:N$44: 7SEG:7SEG.5, 7SEG:R9.2
- new net 7SEG:N$45: 7SEG:7SEGLATCH.12, 7SEG:R9.1
- new net 7SEG:N$5: 7SEG:7SEGLATCH.17, 7SEG:R4.1
- new net 7SEG:N$6: 7SEG:7SEGLATCH.16, 7SEG:R5.1
- new net 7SEG:N$7: 7SEG:7SEGLATCH.15, 7SEG:R6.1
- new net 7SEG:N$8: 7SEG:7SEGLATCH.14, 7SEG:R7.1
- new net 7SEG:N$9: 7SEG:7SEGLATCH.13, 7SEG:R8.1
- new net 7SEGCSWR: 7SEG:7SEGLATCH.11, CSLOGIC100.23
- new net ALE: MC:DEMULTIPLEXER.11, MC:MICROCONTROLLER.30, RTC:RTC.3
- new net MC:N$15: MC:C1.2, MC:MICROCONTROLLER.9, MC:R1.2, MC:RSTSWITCH.1
- new net MC:N$18: MC:JPM.1, MC:MICROCONTROLLER.10
- new net MC:N$19: MC:JPM.2, MC:MICROCONTROLLER.11
- new net MC:N$20: MC:JPM.3, MC:MICROCONTROLLER.12
- new net MC:N$21: MC:JPM.4, MC:MICROCONTROLLER.13
- new net MC:N$22: MC:JPM.5, MC:MICROCONTROLLER.14
- new net MC:N$31: MC:MICROCONTROLLER.18
- new net P3.5: CSLOGIC100.8, MC:MICROCONTROLLER.15
- new net PSEN: CSLOGIC100.2, MC:MICROCONTROLLER.29
- new net PWR:N$2: PWR:PWRFUSE.1A, PWR:S1.3
- new net PWR:N$30: PWR:S1.1
- new net PWR:N$48: PWR:PWRJACK.3, PWR:S1.2
- new net PWR:N$49: PWR:PWRLED.K, PWR:R11.2
- new net RD: ADC:ADC.8, CSLOGIC100.7, MC:MICROCONTROLLER.17, RAM:RAM1.22, RAM:RAM2.22, RTC:RTC.8
- new net WR: ADC:ADC.6, CSLOGIC100.6, MC:MICROCONTROLLER.16, RAM:RAM1.27, RAM:RAM2.27, RTC:RTC.10
- net A0: now also MC:DEMULTIPLEXER.12; no longer MICROCONTROLLER1:DEMULTIPLEXER.12
- net A1: now also MC:DEMULTIPLEXER.13; no longer MICROCONTROLLER1:DEMULTIPLEXER.13
- net A10: now also MC:MICROCONTROLLER.23; no longer MICROCONTROLLER1:MICROCONTROLLER.23
- net A11: now also MC:MICROCONTROLLER.24; no longer MICROCONTROLLER1:MICROCONTROLLER.24
- net A12: now also MC:MICROCONTROLLER.25; no longer MICROCONTROLLER1:MICROCONTROLLER.25
- net A13: now also MC:MICROCONTROLLER.26; no longer MICROCONTROLLER1:MICROCONTROLLER.26
- net A14: now also MC:MICROCONTROLLER.27; no longer MICROCONTROLLER1:MICROCONTROLLER.27
- net A15: now also MC:MICROCONTROLLER.28; no longer MICROCONTROLLER1:MICROCONTROLLER.28
- net A2: now also MC:DEMULTIPLEXER.14; no longer MICROCONTROLLER1:DEMULTIPLEXER.14
- net A3: now also MC:DEMULTIPLEXER.15; no longer MICROCONTROLLER1:DEMULTIPLEXER.15
- net A4: now also MC:DEMULTIPLEXER.16; no longer MICROCONTROLLER1:DEMULTIPLEXER.16
- net A5: now also MC:DEMULTIPLEXER.17; no longer MICROCONTROLLER1:DEMULTIPLEXER.17
- net A6: now also MC:DEMULTIPLEXER.18; no longer MICROCONTROLLER1:DEMULTIPLEXER.18
- net A7: now also MC:DEMULTIPLEXER.19; no longer MICROCONTROLLER1:DEMULTIPLEXER.19
- net A8: now also MC:MICROCONTROLLER.21; no longer MICROCONTROLLER1:MICROCONTROLLER.21
- net A9: now also MC:MICROCONTROLLER.22; no longer MICROCONTROLLER1:MICROCONTROLLER.22
- net ADC:N$26: now also ADC:C2.1
- net D0: now also 7SEG:7SEGLATCH.2, MC:DEMULTIPLEXER.2, MC:MICROCONTROLLER.39; no longer 7SEGDISPLAY:7SEGLATCH.2, MICROCONTROLLER1:DEMULTIPLEXER.2, MICROCONTROLLER1:MICROCONTROLLER.39
- net D1: now also 7SEG:7SEGLATCH.3, MC:DEMULTIPLEXER.3, MC:MICROCONTROLLER.38; no longer 7SEGDISPLAY:7SEGLATCH.3, MICROCONTROLLER1:DEMULTIPLEXER.3, MICROCONTROLLER1:MICROCONTROLLER.38
- net D2: now also 7SEG:7SEGLATCH.4, MC:DEMULTIPLEXER.4, MC:MICROCONTROLLER.37; no longer 7SEGDISPLAY:7SEGLATCH.4, MICROCONTROLLER1:DEMULTIPLEXER.4, MICROCONTROLLER1:MICROCONTROLLER.37
- net D3: now also 7SEG:7SEGLATCH.5, MC:DEMULTIPLEXER.5, MC:MICROCONTROLLER.36; no longer 7SEGDISPLAY:7SEGLATCH.5, MICROCONTROLLER1:DEMULTIPLEXER.5, MICROCONTROLLER1:MICROCONTROLLER.36
- net D4: now also 7SEG:7SEGLATCH.6, MC:DEMULTIPLEXER.6, MC:MICROCONTROLLER.35; no longer 7SEGDISPLAY:7SEGLATCH.6, MICROCONTROLLER1:DEMULTIPLEXER.6, MICROCONTROLLER1:MICROCONTROLLER.35
- net D5: now also 7SEG:7SEGLATCH.7, MC:DEMULTIPLEXER.7, MC:MICROCONTROLLER.34; no longer 7SEGDISPLAY:7SEGLATCH.7, MICROCONTROLLER1:DEMULTIPLEXER.7, MICROCONTROLLER1:MICROCONTROLLER.34
- net D6: now also 7SEG:7SEGLATCH.8, MC:DEMULTIPLEXER.8, MC:MICROCONTROLLER.33; no longer 7SEGDISPLAY:7SEGLATCH.8, MICROCONTROLLER1:DEMULTIPLEXER.8, MICROCONTROLLER1:MICROCONTROLLER.33
- net D7: now also 7SEG:7SEGLATCH.9, MC:DEMULTIPLEXER.9, MC:MICROCONTROLLER.32; no longer 7SEGDISPLAY:7SEGLATCH.9, MICROCONTROLLER1:DEMULTIPLEXER.9, MICROCONTROLLER1:MICROCONTROLLER.32
- net GND: now also 7SEG:7SEGLATCH.1, 7SEG:7SEGLATCH.10, 7SEG:C1.2, ADC:C1.2, ADC:C2.2, C101.2, CLK:CLK.4, CSLOGIC100.12, LCD:C1.2, LCD:C2.2, MC:C2.2, MC:DEMULTIPLEXER.1, MC:DEMULTIPLEXER.10, MC:MICROCONTROLLER.20, MC:MICROCONTROLLER.31, MC:R1.1, PWR:PWRJACK.1, PWR:PWRJACK.2, PWR:R11.1, RAM:C1.2, RAM:C2.2, ROM:C1.2, ROM:C2.2, RTC:C1.2; no longer 7SEGDISPLAY:7SEGLATCH.1, 7SEGDISPLAY:7SEGLATCH.10, CLOCK:CLK.4, MICROCONTROLLER1:DEMULTIPLEXER.1, MICROCONTROLLER1:DEMULTIPLEXER.10, MICROCONTROLLER1:MICROCONTROLLER.20, MICROCONTROLLER1:MICROCONTROLLER.31, MICROCONTROLLER1:R1.1, POWERSP:J1.1, POWERSP:J1.2, POWERSP:R11.1
- net N$5: now also CLK:CLK.5, MC:MICROCONTROLLER.19; no longer CLOCK:CLK.5, MICROCONTROLLER1:MICROCONTROLLER.19
- net PONE0: now also KP:KEYPAD.1, MC:MICROCONTROLLER.1; no longer KEYPAD1:KEYPAD.1, MICROCONTROLLER1:MICROCONTROLLER.1
- net PONE1: now also KP:KEYPAD.2, MC:MICROCONTROLLER.2; no longer KEYPAD1:KEYPAD.2, MICROCONTROLLER1:MICROCONTROLLER.2
- net PONE2: now also KP:KEYPAD.3, MC:MICROCONTROLLER.3; no longer KEYPAD1:KEYPAD.3, MICROCONTROLLER1:MICROCONTROLLER.3
- net PONE3: now also KP:KEYPAD.4, MC:MICROCONTROLLER.4; no longer KEYPAD1:KEYPAD.4, MICROCONTROLLER1:MICROCONTROLLER.4
- net PONE4: now also KP:KEYPAD.5, MC:MICROCONTROLLER.5; no longer KEYPAD1:KEYPAD.5, MICROCONTROLLER1:MICROCONTROLLER.5
- net PONE5: now also KP:KEYPAD.6, MC:MICROCONTROLLER.6; no longer KEYPAD1:KEYPAD.6, MICROCONTROLLER1:MICROCONTROLLER.6
- net PONE6: now also KP:KEYPAD.7, MC:MICROCONTROLLER.7; no longer KEYPAD1:KEYPAD.7, MICROCONTROLLER1:MICROCONTROLLER.7
- net PONE7: now also KP:KEYPAD.8, MC:MICROCONTROLLER.8; no longer KEYPAD1:KEYPAD.8, MICROCONTROLLER1:MICROCONTROLLER.8
- net VCC: now also 7SEG:7SEG.3, 7SEG:7SEG.8, 7SEG:7SEGLATCH.20, 7SEG:C1.1, ADC:C1.1, C101.1, CLK:CLK.8, CSLOGIC100.24, LCD:C1.1, LCD:C2.1, MC:C1.1, MC:C2.1, MC:DEMULTIPLEXER.20, MC:MICROCONTROLLER.40, MC:RSTSWITCH.3, PWR:PWRFUSE.2A, PWR:PWRLED.A, RAM:C1.1, RAM:C2.1, ROM:C1.1, ROM:C2.1, RTC:C1.1; no longer 7SEGDISPLAY:7SEG.3, 7SEGDISPLAY:7SEG.8, 7SEGDISPLAY:7SEGLATCH.20, CLOCK:CLK.8, MICROCONTROLLER1:C1.1, MICROCONTROLLER1:DEMULTIPLEXER.20, MICROCONTROLLER1:MICROCONTROLLER.40, MICROCONTROLLER1:RSTSWITCH.3, POWERSP:LED1.A, POWERSP:S1.3
Routing:
- net VCC: track 0.00 -> 452.0 mm
- net MC:N$15: track 0.00 -> 14.3 mm
- net PWR:N$48: track 0.00 -> 9.00 mm
- net PWR:N$2: track 0.00 -> 8.48 mm
- net PWR:N$49: track 0.00 -> 3.81 mm
Other:
- board size 160 x 100 mm -> 221 x 194.3 mm

Commit message: I made updates to the board and pcb not sure what exactly nothing major
Parts:
- added MC:C3: 0.1uF, Fuckboiz:CAP-PTH-SMALL-KIT
- moved PWR:PWRFUSE 2.54 mm to (39.4, 186.7)
- moved PWR:PWRJACK 2.54 mm to (-2.54, 184.2)
- moved PWR:PWRLED 2.54 mm to (54.6, 186.7)
- moved PWR:R11 2.54 mm to (55.9, 179.1)
- moved PWR:S1 2.54 mm to (26.7, 184.2)
- moved LCD:C1 1.27 mm to (27.9, 91.4)
- moved ROM:ROM1 1.27 mm to (27.9, 110.5)
- moved ROM:ROM2 1.27 mm to (27.9, 45.7)
- moved RTC:C1 1.27 mm to (27.9, 156.2)
Connections:
- net GND: now also MC:C3.2
- net VCC: now also MC:C3.1
Routing:
- net VCC: track 452.0 -> 773.4 mm
- net D6: track 0.00 -> 25.4 mm
- net D5: track 0.00 -> 25.4 mm
- net D4: track 0.00 -> 25.4 mm
- net D3: track 0.00 -> 25.4 mm
- net D2: track 0.00 -> 25.4 mm
- net D1: track 0.00 -> 25.4 mm
- net D0: track 0.00 -> 25.4 mm
- net ADC:N$26: track 0.00 -> 11.8 mm
- net A12: track 0.00 -> 0.65 mm

Commit message: Continued working on traces for signals, changed output of chip_select
Parts:
- moved MC:JPM 184.9 mm to (119.4, 188.0)
- moved CLK:CLK 39.6 mm to (134.6, 26.7), turned to 90 degrees
- moved C101 36.4 mm to (168.9, 67.3)
- moved CSLOGIC100 36.4 mm to (168.9, 48.3)
- moved MC:MICROCONTROLLER 36.3 mm to (134.6, 68.6)
- moved RAM:C1 36.3 mm to (144.8, 97.8)
- moved ADC:C1 35.1 mm to (97.5, 161.3)
- moved RAM:RAM1 35.1 mm to (96.3, 121.9)
- moved MC:DEMULTIPLEXER 32.8 mm to (168.9, 83.8)
- moved RAM:C2 32.8 mm to (168.9, 100.3)
- moved LCD:C2 32.8 mm to (97.5, 83.8)
- moved RAM:RAM2 32.8 mm to (96.3, 44.5)
- moved 7SEG:7SEGLATCH 29.2 mm to (130.8, 129.5)
- moved 7SEG:R2 29.2 mm to (121.9, 141.0)
- moved 7SEG:R6 29.2 mm to (132.1, 141.0)
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Connections:
- net MC:N$18 renamed MC:RXD
- net MC:N$19 renamed MC:TXD
- net MC:N$20 renamed MC:INT0
- net MC:N$21 renamed MC:INT1
- net MC:N$22 renamed MC:T0
- net 7SEGCSWR: now also CSLOGIC100.22; no longer CSLOGIC100.23
- net A0: now also MC:DEMULTIPLEXER.19; no longer MC:DEMULTIPLEXER.12
- net A1: now also MC:DEMULTIPLEXER.18; no longer MC:DEMULTIPLEXER.13
- net A2: now also MC:DEMULTIPLEXER.17; no longer MC:DEMULTIPLEXER.14
- net A3: now also MC:DEMULTIPLEXER.16; no longer MC:DEMULTIPLEXER.15
- net A4: now also MC:DEMULTIPLEXER.15; no longer MC:DEMULTIPLEXER.16
- net A5: now also MC:DEMULTIPLEXER.14; no longer MC:DEMULTIPLEXER.17
- net A6: now also MC:DEMULTIPLEXER.13; no longer MC:DEMULTIPLEXER.18
- net A7: now also MC:DEMULTIPLEXER.12; no longer MC:DEMULTIPLEXER.19
- net ADCCS: now also CSLOGIC100.19; no longer CSLOGIC100.14
- net P3.5: now also CSLOGIC100.6; no longer CSLOGIC100.8
- net RAM1CS: now also CSLOGIC100.15; no longer CSLOGIC100.16
- net RAM2CS: now also CSLOGIC100.14; no longer CSLOGIC100.15
- net RD: now also CSLOGIC100.8; no longer CSLOGIC100.7
- net ROM1CS: now also CSLOGIC100.17; no longer CSLOGIC100.18
- net ROM2CS: now also CSLOGIC100.16; no longer CSLOGIC100.17
- net RTCCS: now also CSLOGIC100.18; no longer CSLOGIC100.22
- net WR: now also CSLOGIC100.7; no longer CSLOGIC100.6
Routing:
- net VCC: track 773.4 -> 0.00 mm
- net ADCCS: track 0.00 -> 225.1 mm, vias 0 -> 1
- net RTCCS: track 0.00 -> 181.9 mm, vias 0 -> 1
- net PONE0: track 0.00 -> 172.2 mm, vias 0 -> 1
- net PONE1: track 0.00 -> 171.8 mm, vias 0 -> 1
- net PONE2: track 0.00 -> 171.5 mm, vias 0 -> 1
- net PONE3: track 0.00 -> 171.0 mm, vias 0 -> 1
- net PONE4: track 0.00 -> 170.4 mm, vias 0 -> 1
- net PONE5: track 0.00 -> 170.1 mm, vias 0 -> 1
- net PONE7: track 0.00 -> 169.8 mm, vias 0 -> 1
- net PONE6: track 0.00 -> 169.7 mm, vias 0 -> 1
- net ALE: track 0.00 -> 163.4 mm, vias 0 -> 1
- net LCDCS: track 0.00 -> 160.3 mm, vias 0 -> 1
- net MC:T0: track 0.00 -> 144.3 mm, vias 0 -> 1
- net MC:INT1: track 0.00 -> 142.5 mm, vias 0 -> 1
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Other:
- board size 221 x 194.3 mm -> 251.5 x 194.3 mm

Commit message: Continued trace work.
Parts:
- moved LCD:C2 3.66 mm to (94.5, 81.8)
- moved ADC:C1 3.21 mm to (94.5, 160.3)
- moved LCD:C1 2.34 mm to (37.1, 90.4)
- moved RTC:C1 2.27 mm to (37.3, 167.4)
Routing:
- net D3: track 63.6 -> 157.5 mm, vias 0 -> 1
- net D4: track 56.8 -> 148.8 mm, vias 0 -> 1
- net D5: track 58.6 -> 148.9 mm, vias 0 -> 1
- net D6: track 60.5 -> 149.6 mm, vias 0 -> 1
- net D7: track 62.4 -> 150.6 mm, vias 0 -> 1
- net A10: track 0.00 -> 86.2 mm, vias 0 -> 1
- net A11: track 0.00 -> 85.3 mm, vias 0 -> 1
- net A9: track 0.00 -> 83.4 mm, vias 0 -> 1
- net A8: track 0.00 -> 82.5 mm, vias 0 -> 1
- net A13: track 0.00 -> 80.5 mm, vias 0 -> 1
- net ROM1CS: track 6.88 -> 13.9 mm
- net ROM2CS: track 0.00 -> 6.25 mm
- net N$5: track 19.7 -> 23.0 mm

Commit message: Finished routing still needs cleanup
Parts:
- added DRILEGEND: (no value), drilegend:DRILEGEND
- moved MC:R1 16.5 mm to (90.4, 170.9)
- moved MC:C1 16.5 mm to (89.2, 177.3)
- moved MC:RSTSWITCH 16.5 mm to (89.2, 184.9)
- moved ADC:C1 9.14 mm to (85.3, 160.3)
- moved LCD:C2 9.14 mm to (85.3, 81.8)
- moved RAM:RAM1 9.14 mm to (87.1, 121.9)
- moved RAM:RAM2 9.14 mm to (87.1, 44.5)
- moved RAM:C1 1.44 mm to (143.8, 96.8)
Routing:
- net VCC: track 0.00 -> 1137.7 mm, vias 0 -> 2
- net D1: track 59.8 -> 637.1 mm, vias 0 -> 8
- net D0: track 58.7 -> 635.4 mm, vias 0 -> 8
- net D2: track 61.7 -> 635.4 mm, vias 0 -> 5
- net A14: track 0.00 -> 469.2 mm, vias 0 -> 6
- net A1: track 0.00 -> 436.3 mm, vias 0 -> 6
- net D3: track 157.5 -> 586.9 mm, vias 1 -> 4
- net A12: track 0.00 -> 428.8 mm, vias 0 -> 6
- net A0: track 0.00 -> 427.9 mm, vias 0 -> 6
- net A7: track 0.00 -> 412.3 mm, vias 0 -> 5
- net WR: track 0.00 -> 404.8 mm, vias 0 -> 4
- net A6: track 0.00 -> 402.6 mm, vias 0 -> 5
- net A5: track 0.00 -> 393.7 mm, vias 0 -> 5
- net RD: track 0.00 -> 393.3 mm, vias 0 -> 4
- net D7: track 150.6 -> 539.2 mm, vias 1 -> 7
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- added copper zone on layer 16, net GND
Other:
- board text added: "01-16"
- board text added: "01-20"
- board text added: "LAYER-STACK"

Commit message: Double checked connections against breadboard prototype fixed connection issues
Connections:
- net N$5 renamed CLKSIG
Routing:
- net GND: track 10.4 -> 62.7 mm, vias 0 -> 2
- net WR: track 404.8 -> 407.7 mm, vias 4 -> 5
- net RD: track 393.3 -> 390.4 mm
- net 7SEGCSWR: track 132.4 -> 134.5 mm
- net VCC: track 1137.7 -> 1139.4 mm, vias 2 -> 3
- net D3: track 586.9 -> 587.8 mm, vias 4 -> 6
- net CLKSIG: track 23.0 -> 22.3 mm

Commit message: Did a lot of clean up work move the lcd down some to make the mounting holes not so close
Parts:
- removed DRILEGEND: (no value), drilegend:DRILEGEND
- ADC:ADC: value ADC -> TLC0820ACN
- PWR:PWRJACK: value DCpowerjack -> 2.1mm
- moved PWR:PWRLED 7.62 mm to (59.9, 186.2)
- moved PWR:R11 7.62 mm to (61.2, 178.6)
- moved PWR:PWRJACK 3.81 mm to (-1.02, 183.6)
- moved PWR:S1 3.81 mm to (28.2, 183.6)
- moved PWR:PWRFUSE 3.81 mm to (40.9, 186.2)
- moved LCD:LCD 1.80 mm to (200.7, 186.7)
- moved MC:C2 1.52 mm to (26.9, 36.3)
- renumbered 7SEG:7SEG to 7SEG:DISPLAY, C101 to CS:C1, CSLOGIC100 to CS:CSLGC, LCD:IC1 to LCD:COLORLATCH, MC:MICROCONTROLLER to MC:UC
Routing:
- net VCC: track 1139.4 -> 1104.9 mm
- net GND: track 62.7 -> 59.1 mm
- net RTCCS: track 181.9 -> 179.3 mm
- net D3: track 587.8 -> 585.4 mm
- net D2: track 635.4 -> 633.0 mm
- net D7: track 539.2 -> 537.4 mm
- net D4: track 508.7 -> 506.9 mm
- net A1: track 436.3 -> 434.5 mm
- net D6: track 530.4 -> 528.6 mm
- net D5: track 519.8 -> 518.0 mm
- net D1: track 637.1 -> 635.8 mm
- net 7SEGCSWR: track 134.5 -> 135.5 mm
- net LCD:N$23: track 72.1 -> 71.4 mm
- net LCD:N$17: track 72.1 -> 71.4 mm
- net LCD:N$24: track 72.1 -> 71.4 mm
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Other:
- board text added: "CONSTRAST"
- board text added: "INT0"
- board text added: "INT1"
- board text added: "LCD"
- board text added: "RXD"
- board text added: "T0"
- board text added: "TXD"
- board text removed: "01-16"
- board text removed: "01-20"
- board text removed: "LAYER-STACK"
