File: ECEN_4330/PROJECT_V2.sch (EAGLE design)
At the start: 0 parts

Commit message: Double checked connections against breadboard prototype fixed connection issues
Changed lines of the file:
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@@
 <module name="CLOCK" prefix="" dx="30.48" dy="20.32">
 <ports>
-<port name="XTAL1" side="right" coord="7.62" direction="io"/>
 <port name="GND" side="left" coord="-7.62" direction="pwr"/>
 <port name="VCC" side="left" coord="-5.08" direction="pwr"/>
+<port name="CLKOUT" side="right" coord="7.62" direction="io"/>
 </ports>
 <variantdefs>
@@
 <parts>
 <part name="CLK" library="crystal" library_urn="urn:adsk.eagle:library:204" deviceset="XO-" device="8" package3d_urn="urn:adsk.eagle:package:12069/1" value="XC269-ND"/>
-<part name="SUPPLY4" library="supply2" library_urn="urn:adsk.eagle:library:372" deviceset="GND" device=""/>
+<part name="SUPPLY4" library="supply1" library_urn="urn:adsk.eagle:library:371" deviceset="GND" device=""/>
 <part name="SUPPLY10" library="supply1" library_urn="urn:adsk.eagle:library:371" deviceset="VCC" device=""/>
 <part name="FRAME7" library="frames" library_urn="urn:adsk.eagle:library:229" deviceset="LETTER_L" device=""/>
@@
 <instances>
 <instance part="CLK" gate="G$1" x="22.86" y="162.56" rot="R90"/>
-<instance part="SUPPLY4" gate="GND" x="27.94" y="134.62"/>
+<instance part="SUPPLY4" gate="1" x="27.94" y="134.62"/>
 <instance part="SUPPLY10" gate="VCC" x="10.16" y="157.48"/>
 <instance part="FRAME7" gate="G$1" x="0" y="0"/>
@@
 <net name="GND" class="0">
 <segment>
-<pinref part="SUPPLY4" gate="GND" pin="GND"/>
+<pinref part="SUPPLY4" gate="1" pin="GND"/>
 <pinref part="CLK" gate="G$1" pin="GND"/>
 <wire x1="27.94" y1="137.16" x2="27.94" y2="149.86" width="0.1524" layer="91"/>
 </segment>
 </net>
-<net name="XTAL1" class="0">
+<net name="CLKOUT" class="0">
 <segment>
 <pinref part="CLK" gate="G$1" pin="OUT"/>
@@
 </segment>
 </net>
-<net name="N$5" class="0">
-<segment>
-<portref moduleinst="MC" port="XTAL1"/>
-<portref moduleinst="CLK" port="XTAL1"/>
-<wire x1="60.96" y1="127" x2="55.88" y2="127" width="0.1524" layer="91"/>
-</segment>
-</net>
 <net name="ALE" class="0">
 <segment>
@@
 </segment>
 </net>
+<net name="CLKSIG" class="0">
+<segment>
+<portref moduleinst="CLK" port="CLKOUT"/>
+<portref moduleinst="MC" port="XTAL1"/>
+<wire x1="55.88" y1="127" x2="60.96" y2="127" width="0.1524" layer="91"/>
+</segment>
+</net>
