File: Schematics/PROJECT_V2.sch (EAGLE design)
At the start: 0 parts

Commit message: Added git ignore, cleaned up some files, commited project paper (ECEN 4330 Final Paper.pdf), added adjuted bom
Other:
- note added: "1/11"
- note added: "10/11"
- note added: "11/11"
- note added: "2/11"
- note added: "3/11"
- note added: "4/11"
- note added: "5/11"
- note added: "6/11"
- note added: "7/11"
- note added: "8/11"
- note added: "9/11"
- note added: "Microprocessor"
- note removed: "Justin Pachl ECEN 4330 OVERALL SCHEMATIC"
- note removed: "Microcontroller"
